File: mm_mcu.kicad_sch (KiCad schematic)
At the start: 18 parts, among them J1 Conn_ARM_JTAG_SWD_10, U1 STM32F030C8Tx

Commit message: fin tp2
Changed lines of the file:
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@@
   )
   (symbol (lib_id "power:+3.3V") (at 140.97 33.02 0) (unit 1)
-    (in_bom yes) (on_board yes) (dnp no) (fields_autoplaced)
+    (in_bom yes) (on_board yes) (dnp no)
     (property "Reference" "#PWR01" (at 140.97 36.83 0)
       (effects (font (size 1.27 1.27)) hide)
     )
-    (property "Value" "+3.3V" (at 140.97 27.94 0)
+    (property "Value" "+3.3V" (at 142.24 26.67 0)
       (effects (font (size 1.27 1.27)))
     )

Commit message: tp3
Parts:
- removed R7: 100, Resistor_SMD:R_0603_1608Metric, symbol Device:R
- renumbered BOOT0 to BOOT1, C6 to C3, C1 to C4, C2 to C5, C3 to C6, C4 to C7, C5 to C8, J1 to J2, R6 to R2, R8 to R4, R9 to R5, R2 to R6, R3 to R7, R4 to R8, R5 to R9, U1 to U2
Connections:
- net OUT_B1: now also U2.19 (PB1)
