File: mm_motor.kicad_sch (KiCad schematic)
At the start: 1 part, among them M1 N20_encoder

Commit message: fin tp2
Parts:
- added M3: N20_encoder, minimouse:N20_with_encoder, symbol minimouse:N20_w_encoder
Changed lines of the file:
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@@
+    )
+  )
+  (symbol (lib_id "minimouse:N20_w_encoder") (at 185.42 90.17 0) (unit 1)
+    (in_bom yes) (on_board yes) (dnp no) (fields_autoplaced)
+    (property "Reference" "M3" (at 187.96 88.9 0)
+      (effects (font (size 1.27 1.27)) (justify left))
+    )
+    (property "Value" "N20_encoder" (at 187.96 91.44 0)
+      (effects (font (size 1.27 1.27)) (justify left))
+    )
+    (property "Footprint" "minimouse:N20_with_encoder" (at 187.96 86.36 0)
+      (effects (font (size 1.27 1.27)) hide)
+    )
+    (property "Datasheet" "" (at 185.42 90.17 0)
+      (effects (font (size 1.27 1.27)) hide)
+    )
+    (instances
+      (project "minimouse"
+        (path "/d8fa4cba-2469-4231-847f-065b6b829f44/7f113667-692a-4f4d-b16f-621d32f3f136"
+          (reference "M3") (unit 1)
+        )
+        (path "/d8fa4cba-2469-4231-847f-065b6b829f44/3975acd0-18ad-47bc-9ce1-d8c4d864aafe"
+          (reference "M4") (unit 1)
+        )
+      )
     )
   )

Commit message: tp3
Parts:
- removed M3: N20_encoder, minimouse:N20_with_encoder, symbol minimouse:N20_w_encoder
- added C14: 2.2uF, Capacitor_SMD:C_0603_1608Metric, symbol Device:C
- added J3: Conn_01x06, Connector_PinHeader_2.54mm:PinHeader_1x06_P2.54mm_Vertical, symbol Connector_Generic:Conn_01x06
- added R18, R20: 100, Resistor_SMD:R_0603_1608Metric, symbol Device:R
Connections:
- net C1: now also R18.2
- net C2: now also R20.2
- net MA: now also J3.1 (Pin_1)
- net MB: now also J3.6 (Pin_6)
- new net: J3.4 (Pin_4), R20.1
- new net: J3.3 (Pin_3), R18.1
- new net +BATT: C14.1, J3.5 (Pin_5)
- new net GND: C14.2, J3.2 (Pin_2)
Other:
- moved on the sheet: M1
