File: mm_motor_control.kicad_sch (KiCad schematic)
At the start: 0 parts

Commit message: fin tp2
Parts:
- added C10: 1nf, symbol Device:C
- added C11: 2.2µf, symbol Device:C
- added C12: 22µf, symbol Device:C
- added C13: 10nf, symbol Device:C
- added C9: 22nf, symbol Device:C
- added R10, R11: 330mohm, symbol Device:R
- added R12, R13: 10k, symbol Device:R
- added R14: 1kohm, symbol Device:R
- added R15: 47kohm, symbol Device:R
- added R16, R17: 18kohm, symbol Device:R
- added U2: STSPIN240, Package_DFN_QFN:VQFN-16-1EP_3x3mm_P0.5mm_EP1.8x1.8mm, symbol Driver_Motor:STSPIN240
Connections:
- net EN: now also R17.1
- net FAULT: now also C13.1, R17.2, U2.13 (EN/FLT)
- net OUT_A1: now also U2.3 (OUTA1)
- net OUT_A2: now also U2.5 (OUTA2)
- net OUT_B1: now also U2.10 (OUTB1)
- net OUT_B2: now also U2.8 (OUTB2)
- net PHASE_A: now also U2.1 (PHA)
- net PHASE_B: now also U2.15 (PHB)
- net PWM_A: now also U2.2 (PWMA)
- net PWM_B: now also U2.16 (PWMB)
- new net: C9.1, R14.2
- new net: R11.1, U2.9 (SENSEB)
- new net: R12.2, R13.1, U2.11 (REF)
- new net: R14.1, R15.1, U2.12 (TOFF)
- new net: R10.1, U2.4 (SENSEA)
- new net +3.3V: C10.1, R16.1, R16.2, U2.14 (STBY/RESET)
- new net +BATT: R12.1
- new net GND: C10.2, C11.2, C12.2, C13.2, C9.2, R10.2, R11.2, R13.2, R15.2, U2.7 (GND)
- new net VS: C11.1, C12.1, U2.6 (VS)

Commit message: tp3
Parts:
- removed C11: 2.2µf, symbol Device:C
- removed C12: 22µf, symbol Device:C
- removed R10: 330mohm, symbol Device:R
- removed R16: 18kohm, symbol Device:R
- added R3: 330mohm, Resistor_SMD:R_0603_1608Metric, symbol Device:R
- C10: value 1nf -> 2.2µf; footprint (none) -> Capacitor_SMD:C_0603_1608Metric
- C11: renamed from C9; footprint (none) -> Capacitor_SMD:C_0603_1608Metric
- C9: renamed from C13; footprint (none) -> Capacitor_SMD:C_0603_1608Metric
- R10: renamed from R17; footprint (none) -> Resistor_SMD:R_0603_1608Metric
- R12, R13, R14, R15: footprint (none) -> Resistor_SMD:R_0603_1608Metric
- R17: renamed from R11; footprint (none) -> Resistor_SMD:R_0603_1608Metric
- renumbered U2 to U3
Connections:
- net VS is gone; now on net +BATT: U3.6 (VS)
- net +BATT: now also C10.1
- net GND: now also U3.17 (EPAD), R3.2
- net at U3.4 (SENSEA): now also R3.1
- net +3.3V renamed STBY/RESET
- net STBY/RESET: no longer C10.1
Other:
- moved on the sheet: R15, R17
