File: mm_power.kicad_sch (KiCad schematic)
At the start: 1 part, among them J5 Conn_01x02

Commit message: fin tp2
Parts:
- added C7, C8: 1.0µf, symbol Device:C
- added U3: LP5907MFX-3.3, Package_TO_SOT_SMD:SOT-23-5, symbol Regulator_Linear:LP5907MFX-3.3
Connections:
- net +BATT: now also C8.1, U3.1 (IN), U3.3 (EN)
- net GND: now also U3.2 (GND)
- new net: C7.1, U3.5 (OUT)
- new net: C7.2, C8.2
Changed lines of the file:
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@@
   (junction (at 86.36 82.55) (diameter 0) (color 0 0 0 0)
   )
+  (junction (at 86.36 78.74) (diameter 0) (color 0 0 0 0)
+  )
+  (junction (at 143.51 78.74) (diameter 0) (color 0 0 0 0)
+  )
   (junction (at 86.36 95.25) (diameter 0) (color 0 0 0 0)
   )
+  (junction (at 143.51 81.28) (diameter 0) (color 0 0 0 0)
+  )
   (wire (pts (xy 86.36 90.17) (xy 86.36 95.25))
     (stroke (width 0) (type default))
   )
+  (wire (pts (xy 143.51 78.74) (xy 143.51 81.28))
+    (stroke (width 0) (type default))
+  )
+  (wire (pts (xy 86.36 78.74) (xy 143.51 78.74))
+    (stroke (width 0) (type default))
+  )
   (wire (pts (xy 95.25 82.55) (xy 86.36 82.55))
     (stroke (width 0) (type default))
   )
-  (wire (pts (xy 86.36 74.93) (xy 86.36 82.55))
-    (stroke (width 0) (type default))
-  )
   (wire (pts (xy 95.25 86.36) (xy 95.25 82.55))
     (stroke (width 0) (type default))
   )
+  (wire (pts (xy 184.15 78.74) (xy 184.15 82.55))
+    (stroke (width 0) (type default))
+  )
+  (wire (pts (xy 179.07 78.74) (xy 184.15 78.74))
+    (stroke (width 0) (type default))
+  )
+  (wire (pts (xy 143.51 78.74) (xy 163.83 78.74))
+    (stroke (width 0) (type default))
+  )
+  (wire (pts (xy 143.51 88.9) (xy 143.51 95.25))
+    (stroke (width 0) (type default))
+  )
   (wire (pts (xy 95.25 92.71) (xy 95.25 95.25))
     (stroke (width 0) (type default))
@@
     (stroke (width 0) (type default))
   )
+  (wire (pts (xy 143.51 95.25) (xy 184.15 95.25))
+    (stroke (width 0) (type default))
+  )
   (wire (pts (xy 86.36 95.25) (xy 86.36 100.33))
     (stroke (width 0) (type default))
@@
     (stroke (width 0) (type default))
   )
+  (wire (pts (xy 86.36 78.74) (xy 86.36 82.55))
+    (stroke (width 0) (type default))
+  )
   (wire (pts (xy 86.36 82.55) (xy 86.36 87.63))
     (stroke (width 0) (type default))
   )
+  (wire (pts (xy 171.45 88.9) (xy 171.45 91.44))
+    (stroke (width 0) (type default))
+  )
+  (wire (pts (xy 184.15 90.17) (xy 184.15 95.25))
+    (stroke (width 0) (type default))
+  )
+  (wire (pts (xy 86.36 78.74) (xy 86.36 74.93))
+    (stroke (width 0) (type default))
+  )
   (wire (pts (xy 80.01 90.17) (xy 86.36 90.17))
     (stroke (width 0) (type default))
   )
+  (wire (pts (xy 143.51 81.28) (xy 163.83 81.28))
+    (stroke (width 0) (type default))
+  )
+  (symbol (lib_id "Device:C") (at 184.15 86.36 0) (unit 1)
+    (in_bom yes) (on_board yes) (dnp no) (fields_autoplaced)
+    (property "Reference" "C7" (at 187.96 85.09 0)
+      (effects (font (size 1.27 1.27)) (justify left))
+    )
+    (property "Value" "1.0µf" (at 187.96 87.63 0)
+      (effects (font (size 1.27 1.27)) (justify left))
+    )
+    (property "Footprint" "" (at 185.1152 90.17 0)
+      (effects (font (size 1.27 1.27)) hide)
+    )
+    (property "Datasheet" "~" (at 184.15 86.36 0)
+      (effects (font (size 1.27 1.27)) hide)
+    )
+    (pin "1")
+    (pin "2")
+    (instances
+      (project "minimouse"
+        (path "/d8fa4cba-2469-4231-847f-065b6b829f44/3f9b0845-5778-418c-a7a8-03da2392145e"
+          (reference "C7") (unit 1)
+        )
+      )
+    )
+  )
   (symbol (lib_id "power:+BATT") (at 86.36 74.93 0) (unit 1)
-    (in_bom yes) (on_board yes) (dnp no) (fields_autoplaced)
+    (in_bom yes) (on_board yes) (dnp no)
     (property "Reference" "#PWR036" (at 86.36 78.74 0)
       (effects (font (size 1.27 1.27)) hide)
@@
         )
       )
+    )
+  )
+  (symbol (lib_id "power:GND") (at 171.45 91.44 0) (unit 1)
+    (in_bom yes) (on_board yes) (dnp no) (fields_autoplaced)
+    (property "Reference" "#PWR010" (at 171.45 97.79 0)
+      (effects (font (size 1.27 1.27)) hide)
+    )
+    (property "Value" "GND" (at 171.45 96.52 0)
+      (effects (font (size 1.27 1.27)))
+    )
+    (property "Footprint" "" (at 171.45 91.44 0)
+      (effects (font (size 1.27 1.27)) hide)
+    )
+    (property "Datasheet" "" (at 171.45 91.44 0)
+      (effects (font (size 1.27 1.27)) hide)
+    )
+    (pin "1")
+    (instances
+      (project "minimouse"
+        (path "/d8fa4cba-2469-4231-847f-065b6b829f44/3f9b0845-5778-418c-a7a8-03da2392145e"
+          (reference "#PWR010") (unit 1)
+        )
+      )
+    )
+  )
+  (symbol (lib_id "Regulator_Linear:LP5907MFX-3.3") (at 171.45 81.28 0) (unit 1)
+    (in_bom yes) (on_board yes) (dnp no) (fields_autoplaced)
+    (property "Reference" "U3" (at 171.45 71.12 0)
+      (effects (font (size 1.27 1.27)))
+    )
+    (property "Value" "LP5907MFX-3.3" (at 171.45 73.66 0)
+      (effects (font (size 1.27 1.27)))
+    )
+    (property "Footprint" "Package_TO_SOT_SMD:SOT-23-5" (at 171.45 72.39 0)
+      (effects (font (size 1.27 1.27)) hide)
+    )
+    (property "Datasheet" "http://www.ti.com/lit/ds/symlink/lp5907.pdf" (at 171.45 68.58 0)
+      (effects (font (size 1.27 1.27)) hide)
+    )
+    (pin "5")
+    (pin "3")
+    (pin "4")
+    (pin "1")
+    (pin "2")
+    (instances
+      (project "minimouse"
+        (path "/d8fa4cba-2469-4231-847f-065b6b829f44/3f9b0845-5778-418c-a7a8-03da2392145e"
+          (reference "U3") (unit 1)
+        )
+      )
+    )
+  )
+  (symbol (lib_id "Device:C") (at 143.51 85.09 0) (unit 1)
+    (in_bom yes) (on_board yes) (dnp no) (fields_autoplaced)
+    (property "Reference" "C8" (at 147.32 83.82 0)
+      (effects (font (size 1.27 1.27)) (justify left))
+    )
+    (property "Value" "1.0µf" (at 147.32 86.36 0)
+      (effects (font (size 1.27 1.27)) (justify left))
+    )
+    (property "Footprint" "" (at 144.4752 88.9 0)
+      (effects (font (size 1.27 1.27)) hide)
+    )
+    (property "Datasheet" "~" (at 143.51 85.09 0)
+      (effects (font (size 1.27 1.27)) hide)
+    )
+    (pin "2")
+    (pin "1")
+    (instances
+      (project "minimouse"
+        (path "/d8fa4cba-2469-4231-847f-065b6b829f44/3f9b0845-5778-418c-a7a8-03da2392145e"
+          (reference "C8") (unit 1)
+        )
+      )

Commit message: tp3
Parts:
- added D1: LED, LED_SMD:LED_0603_1608Metric, symbol Device:LED
- added R11: 330, Resistor_SMD:R_0603_1608Metric, symbol Device:R
- C1: renamed from C8; footprint (none) -> Capacitor_SMD:C_0603_1608Metric
- C2: renamed from C7; footprint (none) -> Capacitor_SMD:C_0603_1608Metric
- renumbered J5 to J1, U3 to U1
Connections:
- net +3.3V: now reaches C2.1, U1.5 (OUT)
- net +3.3V: now also R11.1
- net at C1.2, C2.2: now also D1.1 (K)
- new net: D1.2 (A), R11.2
Other:
- moved on the sheet: C2
