File: minimouse.kicad_pcb (KiCad board)
At the start: 2 copper layers, 90 x 85 mm, 22 parts, among them J1 Conn_ARM_JTAG_SWD_10, J5 Conn_01x02, M1 N20_encoder, M2 N20_encoder, U1 STM32F030C8Tx, U4 HC-SR04

Commit message: tp3
Parts:
- removed the R7 at (152.1, 99.5)
- added C1: 1.0µf, Capacitor_SMD:C_0603_1608Metric, F.Cu at (120.6, 69.5)
- added C10: 2.2µf, Capacitor_SMD:C_0603_1608Metric, F.Cu at (126.4, 98.1)
- added C11: 22nf, Capacitor_SMD:C_0603_1608Metric, F.Cu at (125.9, 89.4)
- added C14: 2.2uF, Capacitor_SMD:C_0603_1608Metric, F.Cu at (126.3, 93.2)
- added C15: 2.2uF, Capacitor_SMD:C_0603_1608Metric, F.Cu at (142.0, 99.1)
- added C16: 2.2uF, Capacitor_SMD:C_0603_1608Metric, F.Cu at (179.8, 92.8)
- added C17: 2.2uF, Capacitor_SMD:C_0603_1608Metric, F.Cu at (156.8, 66.8)
- added C2: 1.0µf, Capacitor_SMD:C_0603_1608Metric, F.Cu at (132.7, 70.2)
- added C9: 10nf, Capacitor_SMD:C_0603_1608Metric, F.Cu at (118.6, 94.6)
- added D1: LED, LED_SMD:LED_0603_1608Metric, F.Cu at (138.5, 72.4)
- added J3: Conn_01x06, Connector_PinHeader_2.54mm:PinHeader_1x06_P2.54mm_Vertical, F.Cu at (185.8, 82.4)
- added J4: Conn_01x06, Connector_PinHeader_2.54mm:PinHeader_1x06_P2.54mm_Vertical, F.Cu at (116.2, 74.9)
- added J5: Conn_01x04, Connector_PinHeader_2.54mm:PinHeader_1x04_P2.54mm_Vertical, F.Cu at (173.9, 94.3)
- added R10: 18kohm, Resistor_SMD:R_0603_1608Metric, F.Cu at (110.2, 93.0)
- added R11: 330, Resistor_SMD:R_0603_1608Metric, F.Cu at (133.5, 72.8)
- added R12: 10k, Resistor_SMD:R_0603_1608Metric, F.Cu at (126.5, 95.6)
- added R13: 10k, Resistor_SMD:R_0603_1608Metric, F.Cu at (126.8, 101.4)
- added R14: 1kohm, Resistor_SMD:R_0603_1608Metric, F.Cu at (136.1, 83.6)
- added R15: 47kohm, Resistor_SMD:R_0603_1608Metric, F.Cu at (135.4, 76.9)
- added R17: 330mohm, Resistor_SMD:R_0603_1608Metric, F.Cu at (131.4, 92.3)
- added R18: 100, Resistor_SMD:R_0603_1608Metric, F.Cu at (143.2, 69.0)
- added R19: 100, Resistor_SMD:R_0603_1608Metric, F.Cu at (142.1, 77.8)
- added R20: 100, Resistor_SMD:R_0603_1608Metric, F.Cu at (174.1, 82.0)
- added R21: 100, Resistor_SMD:R_0603_1608Metric, F.Cu at (127.3, 84.3)
- added R22: 100, Resistor_SMD:R_0603_1608Metric, F.Cu at (160.5, 79.6)
- added R23: 100, Resistor_SMD:R_0603_1608Metric, F.Cu at (156.2, 72.0)
- added R3: 330mohm, Resistor_SMD:R_0603_1608Metric, F.Cu at (141.3, 95.8)
- added U1: LP5907MFX-3.3, Package_TO_SOT_SMD:SOT-23-5, F.Cu at (128.1, 67.2)
- added U3: STSPIN240, Package_DFN_QFN:VQFN-16-1EP_3x3mm_P0.5mm_EP1.8x1.8mm, F.Cu at (133.2, 97.2)
- moved J1 66.8 mm to (124.5, 73.6), turned to 0 degrees
- moved C8 62.2 mm to (184.8, 75.1), turned to -90 degrees
- moved C6 36.5 mm to (177.2, 75.1), turned to -90 degrees
- moved C7 31.2 mm to (180.5, 75.2), turned to 90 degrees
- moved C4 30.4 mm to (168.1, 75.0), turned to 90 degrees
- moved C5 28.8 mm to (172.8, 75.0)
- moved R7 23.2 mm to (162.4, 86.6), turned to 0 degrees
- moved R6 22.7 mm to (162.3, 84.8), turned to 0 degrees
- moved C3 22.3 mm to (164.4, 75.0)
- moved R8 20.7 mm to (162.3, 88.7), turned to 0 degrees
- moved R9 18.7 mm to (163.0, 91.5), turned to 0 degrees
- moved R2 16.4 mm to (143.2, 84.8), turned to 180 degrees
- moved J2 14.4 mm to (157.9, 96.3)
- moved BOOT1 11.6 mm to (161.7, 67.5)
- moved R4 10.4 mm to (143.3, 87.7), turned to 0 degrees
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- renumbered BOOT0 to BOOT1, C6 to C3, C1 to C4, C2 to C5, C3 to C6, C4 to C7, C5 to C8, J5 to J1, J1 to J2, M2 to M3, R6 to R2, R8 to R4, R9 to R5, R2 to R6, R3 to R7, R4 to R8, R5 to R9, U1 to U2
Connections:
- U2 pad 19: Net-(U1-PB1) -> /mcu/OUT_B1
- U2 pad 43: /mcu/UART1_RX -> /external_uart/EXT_UART_TX
- U4 pad 4: +3V3 -> +3.3V

Commit message: tp3 1
Parts:
- moved R10 40.7 mm to (150.8, 94.9)
- moved R18 38.8 mm to (179.7, 82.2), turned to 90 degrees
- moved C11 37.7 mm to (162.7, 97.5), turned to 180 degrees
- moved C10 34.1 mm to (160.2, 102.5)
- moved R14 31.3 mm to (162.7, 100.0)
- moved C9 29.0 mm to (147.5, 92.4), turned to 90 degrees
- moved R13 28.9 mm to (155.1, 95.7)
- moved R12 28.6 mm to (155.1, 97.5), turned to 180 degrees
- moved R5 28.1 mm to (167.9, 77.1), turned to 180 degrees
- moved R17 24.9 mm to (155.1, 100.0)
- moved R4 24.0 mm to (165.9, 79.7), turned to 180 degrees
- moved R19 22.8 mm to (119.5, 74.6), turned to 180 degrees
- moved J5 22.3 mm to (172.9, 72.1), turned to 90 degrees
- moved R22 21.6 mm to (177.9, 67.0), turned to 90 degrees
- moved C8 21.4 mm to (163.4, 75.4), turned to 90 degrees
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Routing:
- net GND: track 0.00 -> 177.8 mm
- net +BATT: track 0.00 -> 92.1 mm
- net +3.3V: track 0.00 -> 81.9 mm
- net /mcu/IN_B2: track 0.00 -> 32.8 mm
- net /mcu/OUT_B9: track 0.00 -> 28.3 mm
- net Net-(U4-ECHO): track 0.00 -> 20.0 mm
- net Net-(U2-PB9): track 0.00 -> 14.1 mm
- net /mcu/OUT_B1: track 0.00 -> 12.5 mm
- net /mcu/BOOT0: track 0.00 -> 11.6 mm
- net Net-(J4-Pin_3): track 0.00 -> 9.50 mm
- net Net-(D1-K): track 0.00 -> 9.40 mm
- net Net-(U2-PB6): track 0.00 -> 9.09 mm
- net Net-(U3-REF): track 0.00 -> 7.41 mm
- net Net-(U2-PB0): track 0.00 -> 7.28 mm
- net Net-(J3-Pin_3): track 0.00 -> 6.25 mm
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